Commit message: added implementation of laser_filters package
includes custom laser filter node -min value filter and median filter
added use of laser_filter in a separate node
integrated in a single launch file
by using launch arguments, we can run each method

File: task2_ws/src/tortoisebot_description/models/tortoisebot_Task2.urdf (robot description, URDF)
Before this commit: robot tortoisebot, 6 links, 5 joints
Joints:
- joint lidar_joint: origin xyz=0 0 0.180 rpy=0 3.14 0 -> xyz=0 0 0.180 rpy=0 0 0
